File: Eagle/smartFootballTable_ver1.brd (EAGLE design)
At the start: 97.8 x 47 mm, 22 parts, among them IC1 LM2940CT, K1 ARK500/2

Commit message: Updated board with latest changes after soldering
Parts:
- removed J5: (no value), jumper:04C
- added JP1: (no value), jumper:JP2W
Connections:
- net +5V: now also JP1.1; no longer J5.1
- net GND: now also JP1.3; no longer J5.3
- net N$31: now also JP1.2; no longer J5.2
Routing:
- net N$1: track 21.5 -> 16.8 mm
- net N$5: track 48.9 -> 50.6 mm
- net N$31: track 11.5 -> 10.6 mm
- net +5V: track 185.5 -> 186.3 mm
Changed lines of the file:
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@@
 <wire x1="0" y1="46.99" x2="0" y2="0" width="0.3048" layer="20"/>
 <circle x="49.53" y="8.89" radius="8.51941875" width="0.3048" layer="21"/>
-<hole x="3.81" y="44.45" drill="2.2"/>
-<hole x="3.81" y="2.54" drill="2.2"/>
-<hole x="93.98" y="44.45" drill="2.2"/>
+<hole x="3.81" y="44.45" drill="3.2"/>
+<hole x="3.81" y="2.54" drill="3.2"/>
+<hole x="93.98" y="44.45" drill="3.2"/>
 <text x="6.35" y="2.54" size="1.016" layer="25">Smart Football Table</text>
 <text x="6.35" y="1.27" size="1.016" layer="25">ver.1</text>
@@
 <attribute name="VALUE" x="97.79" y="19.05" size="1.27" layer="27" rot="R180"/>
 </element>
-<element name="J5" library="jumper" package="04C" value="" x="48.26" y="33.02" rot="R180"/>
 <element name="K1" library="#PaJa_konektory" package="ARK500/2" value="ARK500/2" x="90.17" y="3.81" smashed="yes">
 <attribute name="NAME" x="84.138" y="2.385" size="1.4224" layer="25" rot="R90"/>
@@
 <attribute name="VALUE" x="67.7908" y="7.942" size="1.27" layer="27" rot="R180"/>
 </element>
+<element name="JP1" library="jumper" package="JP2W" value="" x="45.5461125" y="32.339428125" rot="R180"/>
 </elements>
 <signals>
@@
 <contactref element="SENS_1" pad="6"/>
 <contactref element="SENS_1" pad="7"/>
-<contactref element="J5" pad="3"/>
 <contactref element="SENS_2" pad="6"/>
 <contactref element="SENS_2" pad="7"/>
@@
 <wire x1="40.64" y1="39.37" x2="40.64" y2="45.6692" width="0.3048" layer="16"/>
 <wire x1="67.31" y1="40.64" x2="67.31" y2="33.02" width="0.3048" layer="16"/>
-<wire x1="40.64" y1="34.29" x2="41.91" y2="33.02" width="0.3048" layer="16"/>
-<wire x1="41.91" y1="33.02" x2="42.545" y2="33.02" width="0.3048" layer="16"/>
 <wire x1="40.64" y1="45.6692" x2="45.72" y2="45.6692" width="0.3048" layer="16"/>
 <wire x1="45.72" y1="45.6692" x2="87.63" y2="45.6692" width="0.3048" layer="16"/>
@@
 <vertex x="-1.27" y="-1.27"/>
 </polygon>
+<contactref element="JP1" pad="3"/>
+<wire x1="40.64" y1="34.29" x2="41.320571875" y2="33.609428125" width="0.3048" layer="16"/>
+<wire x1="41.320571875" y1="33.609428125" x2="43.0061125" y2="33.609428125" width="0.3048" layer="16"/>
 </signal>
 <signal name="VIN">
@@
 <contactref element="DIS_1" pad="1"/>
 <contactref element="DIS_2" pad="1"/>
-<contactref element="J5" pad="1"/>
 <contactref element="SENS_1" pad="1"/>
 <wire x1="12.7" y1="25.4" x2="8.89" y2="25.4" width="0.3048" layer="1"/>
@@
 <wire x1="10.16" y1="6.35" x2="12.7" y2="6.35" width="0.3048" layer="1"/>
 <wire x1="38.1" y1="35.56" x2="47.625" y2="35.56" width="0.3048" layer="1"/>
-<wire x1="47.625" y1="35.56" x2="50.165" y2="33.02" width="0.3048" layer="1"/>
-<wire x1="50.165" y1="33.02" x2="54.61" y2="33.02" width="0.3048" layer="1"/>
 <wire x1="54.61" y1="33.02" x2="54.61" y2="22.86" width="0.3048" layer="1"/>
 <wire x1="54.61" y1="22.86" x2="57.15" y2="20.32" width="0.3048" layer="1"/>
@@
 <wire x1="66.04" y1="19.05" x2="69.85" y2="22.86" width="0.3048" layer="1"/>
 <wire x1="69.85" y1="22.86" x2="77.47" y2="22.86" width="0.3048" layer="1"/>
+<contactref element="JP1" pad="1"/>
+<wire x1="47.625" y1="35.56" x2="48.0861125" y2="35.0988875" width="0.3048" layer="1"/>
+<wire x1="48.0861125" y1="35.0988875" x2="48.0861125" y2="33.609428125" width="0.3048" layer="1"/>
+<wire x1="48.0861125" y1="33.609428125" x2="48.675540625" y2="33.02" width="0.3048" layer="1"/>
+<wire x1="48.675540625" y1="33.02" x2="54.61" y2="33.02" width="0.3048" layer="1"/>
 </signal>
 <signal name="D12">
@@
 <contactref element="R3" pad="2"/>
 <contactref element="R4" pad="2"/>
-<contactref element="J5" pad="2"/>
-<wire x1="46.355" y1="33.02" x2="46.355" y2="33.655" width="0.3048" layer="16"/>
-<wire x1="46.355" y1="33.655" x2="43.18" y2="36.83" width="0.3048" layer="16"/>
-<wire x1="43.18" y1="36.83" x2="43.18" y2="39.37" width="0.3048" layer="16"/>
+<wire x1="43.18" y1="39.37" x2="43.18" y2="36.83" width="0.3048" layer="16"/>
 <wire x1="43.18" y1="39.37" x2="43.18" y2="43.18" width="0.3048" layer="16"/>
+<contactref element="JP1" pad="2"/>
+<wire x1="43.18" y1="36.83" x2="45.5461125" y2="34.4638875" width="0.3048" layer="16"/>
+<wire x1="45.5461125" y1="34.4638875" x2="45.5461125" y2="33.609428125" width="0.3048" layer="16"/>
 </signal>
 <signal name="N$1">
@@
 <contactref element="K1" pad="1"/>
 <contactref element="J1" pad="1"/>
-<wire x1="90.63" y1="12.7" x2="92.71" y2="10.62" width="0.6096" layer="16"/>
-<wire x1="92.71" y1="7.62" x2="92.71" y2="10.62" width="0.6096" layer="16"/>
-<wire x1="87.63" y1="7.62" x2="80.9625" y2="7.62" width="0.6096" layer="16"/>
-<wire x1="87.63" y1="7.62" x2="92.71" y2="7.62" width="0.6096" layer="16"/>
-<wire x1="87.63" y1="3.81" x2="87.63" y2="7.62" width="0.8128" layer="16"/>
+<wire x1="90.63" y1="12.7" x2="87.63" y2="9.7" width="1.016" layer="16"/>
+<wire x1="87.63" y1="7.6192375" x2="87.63" y2="9.7" width="1.016" layer="16"/>
+<wire x1="87.63" y1="7.6192375" x2="87.63" y2="3.81" width="1.016" layer="16"/>
+<wire x1="80.9625" y1="7.62" x2="80.9632625" y2="7.6192375" width="1.016" layer="16"/>
+<wire x1="80.9632625" y1="7.6192375" x2="87.63" y2="7.6192375" width="1.016" layer="16"/>
 </signal>
 <signal name="N$5">
@@
 <contactref element="J1" pad="3"/>
 <contactref element="J1" pad="2"/>
-<wire x1="87.63" y1="12.7" x2="87.63" y2="17.5" width="0.6096" layer="16"/>
-<wire x1="87.63" y1="12.7" x2="84.63" y2="12.7" width="0.6096" layer="16"/>
-<wire x1="87.63" y1="17.5" x2="87.91" y2="17.78" width="0.6096" layer="16"/>
-<wire x1="87.91" y1="17.78" x2="92.71" y2="17.78" width="0.6096" layer="16"/>
-<wire x1="92.71" y1="17.78" x2="95.25" y2="15.24" width="0.6096" layer="16"/>
-<wire x1="95.25" y1="7.62" x2="95.25" y2="15.24" width="0.6096" layer="16"/>
+<wire x1="87.91" y1="17.78" x2="87.63" y2="17.5" width="0.6096" layer="16"/>
 <wire x1="74.93" y1="2.54" x2="74.93" y2="1.4732" width="0.6096" layer="16"/>
 <wire x1="92.71" y1="3.81" x2="92.71" y2="5.08" width="0.8128" layer="16"/>
-<wire x1="92.71" y1="5.08" x2="95.25" y2="7.62" width="0.8128" layer="16"/>
 <wire x1="90.3732" y1="1.4732" x2="92.71" y2="3.81" width="0.3048" layer="16"/>
 <wire x1="74.93" y1="1.4732" x2="90.3732" y2="1.4732" width="0.3048" layer="16"/>
+<wire x1="84.63" y1="12.7" x2="87.63" y2="15.7" width="1.016" layer="16"/>
+<wire x1="87.63" y1="15.7" x2="87.63" y2="17.5" width="1.016" layer="16"/>
+<wire x1="87.63" y1="17.5" x2="87.8235625" y2="17.6935625" width="1.016" layer="16"/>
+<wire x1="87.8235625" y1="17.6935625" x2="95.57910625" y2="17.6935625" width="1.016" layer="16"/>
+<wire x1="95.57910625" y1="17.6935625" x2="95.49445" y2="17.60890625" width="1.016" layer="16"/>
+<wire x1="95.49445" y1="17.60890625" x2="95.49445" y2="6.603340625" width="1.016" layer="16"/>
+<wire x1="95.49445" y1="6.603340625" x2="92.71" y2="3.818890625" width="1.016" layer="16"/>
+<wire x1="92.71" y1="3.818890625" x2="92.71" y2="3.81" width="1.016" layer="16"/>
 </signal>
 </signals>

Commit message: Added pin description and started with PlatformIO
Connections:
- net D10 renamed DIS1_DIO
- net D5 renamed DIS2_CLK
- net D6 renamed DIS2_DIO
- net D7 renamed DIS2_UP
- net D8 renamed DIS2_DOWN
- net D9 renamed DIS1_CLK
Changed lines of the file:
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@@
 <wire x1="16.51" y1="11.43" x2="22.86" y2="10.16" width="0.3048" layer="16"/>
 </signal>
-<signal name="D10">
+<signal name="DIS1_DIO">
 <contactref element="ARDUINO_NANO1" pad="28"/>
 <contactref element="DIS_1" pad="4"/>
@@
 <wire x1="16.51" y1="13.97" x2="22.86" y2="12.7" width="0.3048" layer="16"/>
 </signal>
-<signal name="D9">
+<signal name="DIS1_CLK">
 <contactref element="ARDUINO_NANO1" pad="27"/>
 <contactref element="DIS_1" pad="5"/>
@@
 <wire x1="16.51" y1="16.51" x2="22.86" y2="15.24" width="0.3048" layer="16"/>
 </signal>
-<signal name="D8">
+<signal name="DIS2_DOWN">
 <contactref element="ARDUINO_NANO1" pad="26"/>
 <contactref element="DIS_2" pad="2"/>
@@
 <wire x1="15.24" y1="27.94" x2="12.7" y2="27.94" width="0.3048" layer="16"/>
 </signal>
-<signal name="D7">
+<signal name="DIS2_UP">
 <contactref element="ARDUINO_NANO1" pad="25"/>
 <contactref element="DIS_2" pad="3"/>
@@
 <wire x1="15.24" y1="30.48" x2="12.7" y2="30.48" width="0.3048" layer="16"/>
 </signal>
-<signal name="D6">
+<signal name="DIS2_DIO">
 <contactref element="ARDUINO_NANO1" pad="24"/>
 <contactref element="DIS_2" pad="4"/>
@@
 <wire x1="16.51" y1="33.02" x2="12.7" y2="33.02" width="0.3048" layer="16"/>
 </signal>
-<signal name="D5">
+<signal name="DIS2_CLK">
 <contactref element="ARDUINO_NANO1" pad="23"/>
 <contactref element="DIS_2" pad="5"/>
